File: breakout_board_PCB/BreakoutBoardPCB/BreakoutBoardPCB.kicad_sch (KiCad schematic)
At the start: 65 parts, among them IC1 AD5676BRUZ, J1 USB_B_Micro - 10118193-0001LF, J10 Conn_01x27_Female, J11 Conn_01x20_Female, J2 Conn_01x02_Female, J3 Conn_01x02_Male, J4 Conn_01x03_Female, J5 Conn_01x02_Male, J6 Conn_01x02_Male, J7 Conn_01x06_Female, J8 Conn_01x02_Male, J9 Conn_01x02_Male, SW1 SW_Push - SKQGADE010, T1 Logo, T2 Logo, U1 FT232H, U2 SN74LVC1G125DCKR, U3 SN74LVC1G125DCKR, U4 MCP1319MT-29LE-OT, U5 TAR5SxxU_SOT353F, U6 TAR5SxxU_SOT353F, U7 W25Q32FVSS, U8 caravel-M.2-card, X1 DSC6001_10MHZ, Y1 CSTNE12M0GH5L000R0

Commit message: update
Parts:
- removed C10, C13: 1uf - CC0805KKX5R8BB105, Capacitor_SMD:C_0805_2012Metric, symbol Device:C
- removed C11, C14: 0.01uf - CC0805KRX7R9BB103, Capacitor_SMD:C_0805_2012Metric, symbol Device:C
- removed C12, C15: 10uf - CC0805KKX5R8BB106, Capacitor_SMD:C_0805_2012Metric, symbol Device:C
- removed C16, C17, C5, C6, C7, C8, C9: 0.1uf - CC0805KRX7R9BB104, Capacitor_SMD:C_0805_2012Metric, symbol Device:C
- removed D1, D2, D3, D4: LED - 17-215SURC/S530-A2/TR8, LED_SMD:LED_1206_3216Metric, symbol Device:LED
- removed H1: MICROMOD-Standoff, MicroMod-Sparkfun:MicroMod-Standoff, symbol MicroMod-Sparkfun:MICROMOD-Standoff
- removed J1: USB_B_Micro - 10118193-0001LF, strive_foot_prints:FCI_10118193-0001LF, symbol Connector:USB_B_Micro
- removed J2: Conn_01x02_Female, Connector_PinHeader_2.54mm:PinHeader_1x02_P2.54mm_Vertical, symbol Connector:Conn_01x02_Female
- removed J3, J5, J6, J8, J9: Conn_01x02_Male, Connector_PinHeader_2.54mm:PinHeader_1x02_P2.54mm_Vertical, symbol Connector:Conn_01x02_Male
- removed J4: Conn_01x03_Female, Connector_PinHeader_2.54mm:PinHeader_1x03_P2.54mm_Vertical, symbol Connector:Conn_01x03_Pin
- removed R1, R10, R12, R13, R7, R8, R9: 10k - RC0805FR-0710KL, Resistor_SMD:R_0805_2012Metric, symbol Device:R
- removed R11, R14: 82 - 0805W8F820JT5E, Resistor_SMD:R_0805_2012Metric, symbol Device:R
- removed R15, R16, R5, R6: 10k, Resistor_SMD:R_0805_2012Metric, symbol Device:R
- removed R2: 12K 1% - 0805W8F1202T5E, Resistor_SMD:R_0805_2012Metric, symbol Device:R
- removed R3, R4: 150 - 0805W8J0151T5E, Resistor_SMD:R_0805_2012Metric, symbol Device:R
- removed SW1: SW_Push - SKQGADE010, strive_foot_prints:SW4-SMD-5.2X5.2X1.5MM, symbol Switch:SW_Push
- removed T1: Logo, Caravel_Board:logo, symbol Caravel_board:Logo
- removed T2: Logo, Caravel_Board:ef_logo, symbol Caravel_board:Logo
- removed TP1, TP2: TestPoint, TestPoint:TestPoint_Bridge_Pitch2.54mm_Drill1.0mm, symbol Connector:TestPoint
- removed U1: FT232H, Package_DFN_QFN:QFN-48-1EP_8x8mm_P0.5mm_EP6.2x6.2mm, symbol Interface_USB:FT232H
- removed U2, U3: SN74LVC1G125DCKR, SOT65P210X110-5N, symbol Caravel_board:SN74LVC1G125DCKR
- removed U4: MCP1319MT-29LE-OT, Caravel_Board:PoR_5_SOT23, symbol Caravel_board:MCP1319MT-29LE-OT
- removed U5, U6: TAR5SxxU_SOT353F, Caravel_Board:SOT-353F, symbol Caravel_board:TAR5SxxU_SOT353F
- removed U7: W25Q32FVSS, strive_foot_prints:SOIC127P790X216-8N, symbol Caravel_board:W25Q32FVSS
- removed U8: caravel-M.2-card, MicroMod-Sparkfun:M.2-CONNECTOR-E, symbol Caravel_board:caravel-M.2-card
- removed X1: DSC6001_10MHZ, strive_foot_prints:DSC6001JE1A-010.0000, symbol Oscillator:XO91
- removed Y1: CSTNE12M0GH5L000R0, strive_foot_prints:CSTNE12M0GH5L000R0, symbol Device:Crystal_GND2
- added IC2: ADS1178IPAPT, QFP50P1200X1200X120-65N, symbol SeniorDesign:ADS1178IPAPT
- added IC3, IC4, IC5, IC6: 23K256T-I_SN, SOIC127P600X175-8N, symbol SeniorDesign:23K256T-I_SN
- C1: value 0.01uf - CC0805JRX7R9BB103 -> 0.1uf - CC0805KRX7R9BB104
Connections:
- net +1V8: no longer J11.24 (Pin_24)
- net +3.3V: now also C1.1, C2.1, C3.1, C4.1, IC3.8 (VCC), IC4.8 (VCC), IC5.8 (VCC), IC6.8 (VCC); no longer C4.2, J10.7 (Pin_7)
- net Caravel_CSB: now also IC3.1 (~{CS}), IC4.1 (~{CS}), IC5.1 (~{CS}), IC6.1 (~{CS})
- net Caravel_D0: now also IC3.5 (SI), IC4.5 (SI), IC5.5 (SI), IC6.5 (SI)
- net Caravel_D1: now also IC3.2 (SO), IC4.2 (SO), IC5.2 (SO), IC6.2 (SO)
- net Caravel_SCK: now also IC3.6 (SCK), IC4.6 (SCK), IC5.6 (SCK), IC6.6 (SCK)
- net GND: now also C1.2, C2.2, C3.2, C4.2, IC1.13 (GND), IC1.14 (RSTSEL), IC1.5 (~{SYNC}), IC2.10 (CLKDIV), IC2.11 (~{SYNC}), IC2.12 (DIN), IC2.21 (DGND_2), IC2.24 (DGND_3), IC2.25 (DGND_4), IC2.35 (~{PWDN8}), IC2.36 (~{PWDN7}), IC2.37 (~{PWDN6}), IC2.38 (~{PWDN5}), IC2.39 (~{PWDN4}), IC2.40 (~{PWDN3}), IC2.41 (~{PWDN2}), IC2.42 (~{PWDN1}), IC2.43 (AGND_2), IC2.54 (AGND_3), IC2.58 (AGND_4), IC2.59 (AGND_5), IC2.6 (AGND_1), IC2.7 (DGND_1), IC2.8 (TEST0), IC2.9 (TEST1), IC3.4 (VSS), IC4.4 (VSS), IC5.4 (VSS), IC6.4 (VSS); no longer C1.1, C2.1, C3.1, C4.1
- net mprj_io[14]: now also IC2.34 (MODE)
- net ~{MEM_HOLD}: now also IC3.7 (~{HOLD}), IC4.7 (~{HOLD}), IC5.7 (~{HOLD}), IC6.7 (~{HOLD})
- net ~{RST}: now also IC1.17 (~{RESET})
- net Vref: now reaches IC1.18 (VREF)
- net Vref: now also IC2.55 (VCOM), IC2.56 (VREFP)
- net vddio: now reaches IC1.3 (VDD)
- net vddio: now also J10.7 (Pin_7), IC2.44 (AVDD_2), IC2.5 (AVDD_1), IC2.53 (AVDD_3), IC2.60 (AVDD_4)
- net USB_CS1 renamed mprj_io[3]_CSB
- net USB_SCK_TXD renamed mprj_io[4]_SCK
- net mprj_io[4]_SCK: now also IC2.28 (SCLK)
- net USB_SI renamed mprj_io[1]_SDO
- net USB_SO_RXD renamed mprj_io[2]_SDI
- new net vccd1: IC2.26 (DVDD), J11.24 (Pin_24)
- no-connect marks 26 -> 0
Other:
- note added: "0 = high speed, 1 = low speed"
- note added: "ADC"
- note added: "DAC"
- note added: "SRAM"
- note removed: "Buffers to enable FTDI UART interface"
- note removed: "FTDI Module"
- note removed: "FTDI interface with HKSPI"
- note removed: "Flash memory"
- note removed: "LEDs"
- note removed: "MEMS Oscillator"
- note removed: "Power on Reset"
- note removed: "Serial Display"
- note removed: "USB Module"
- note removed: "Voltage Regulator"
- moved on the sheet: IC1, J10, J11
