File: breakout_board_PCB/BreakoutBoardPCB/BreakoutBoardPCB.kicad_sch (KiCad schematic)
At the start: 13 parts, among them IC1 AD5676BRUZ, IC2 MCP3464T-E_NC, IC3 23K256T-I_SN, IC4 23K256T-I_SN, IC5 23K256T-I_SN, IC6 23K256T-I_SN, J10 Conn_01x27_Female, J11 Conn_01x20_Female, J7 Conn_01x06_Female

Commit message: update
Parts:
- added J1, J2: SJ-63062A, CUI_SJ-63062A, symbol SeniorDesign:SJ-63062A
Connections:
- net GND: now also J1.2, J2.2; no longer IC2.16 (MCLK)
- net mprj_io[14]: now also IC2.16 (MCLK)
- net mprj_io[22]: no longer IC2.3 (CH0)
- net mprj_io[30]: no longer IC1.2 (VOUT0)
- new net: IC1.2 (VOUT0), J2.1
- new net: IC2.3 (CH0), J1.1
Other:
- note added: "input jack"
- note added: "output jack"
