File: breakout_board_PCB/BreakoutBoardPCB/BreakoutBoardPCB.kicad_pcb (KiCad board)
At the start: 2 copper layers, 76.2 x 73.8 mm, 65 parts, among them IC1 AD5676BRUZ, J1 USB_B_Micro - 10118193-0001LF, J10 Conn_01x27_Female, J11 Conn_01x20_Female, J2 Conn_01x02_Female, J3 Conn_01x02_Male, J4 Conn_01x03_Female, J5 Conn_01x02_Male, J6 Conn_01x02_Male, J7 Conn_01x06_Female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

Commit message: test
Parts:
- removed C1: 0.01uf - CC0805JRX7R9BB103, Capacitor_SMD:C_0805_2012Metric
- removed C11: 0.01uf - CC0805KRX7R9BB103, Capacitor_SMD:C_0805_2012Metric
- removed C12: 10uf - CC0805KKX5R8BB106, Capacitor_SMD:C_0805_2012Metric
- removed C2, C3, C4, C5, C6, C7, C8, C9: 0.1uf - CC0805KRX7R9BB104, Capacitor_SMD:C_0805_2012Metric
- removed D1, D2: LED - 17-215SURC/S530-A2/TR8, LED_SMD:LED_1206_3216Metric
- removed J5, J9: Conn_01x02_Male, Connector_PinHeader_2.54mm:PinHeader_1x02_P2.54mm_Vertical
- removed R1: 10k - RC0805FR-0710KL, Resistor_SMD:R_0805_2012Metric
- removed R15: 10k, Resistor_SMD:R_0805_2012Metric
- removed R3, R4: 150 - 0805W8J0151T5E, Resistor_SMD:R_0805_2012Metric
- removed T1: Logo, Caravel_Board:logo
- removed T2: Logo, Caravel_Board:ef_logo
- added IC**: SOIC127P600X175-8N (SRAM), SeniorDesign:SOIC127P600X175-8N (SRAM), F.Cu at (223.5, 129.5)
- added IC**: SOIC127P600X175-8N (SRAM), SeniorDesign:SOIC127P600X175-8N (SRAM), F.Cu at (213.4, 129.5)
- added IC**: SOIC127P600X175-8N (SRAM), SeniorDesign:SOIC127P600X175-8N (SRAM), F.Cu at (223.5, 137.2)
- added IC**: SOIC127P600X175-8N (SRAM), SeniorDesign:SOIC127P600X175-8N (SRAM), F.Cu at (213.4, 137.2)
- added IC**: QFP50P1200X1200X120-65N (ADC), SeniorDesign:QFP50P1200X1200X120-65N (ADC), F.Cu at (190.5, 127.0)
- moved U7 32.4 mm to (186.1, 161.1)
- moved U1 28.2 mm to (179.1, 137.2)
- moved D3 22.6 mm to (148.7, 195.6)
- moved U4 13.3 mm to (114.7, 114.3)
- moved D4 6.32 mm to (123.3, 195.6)
- moved IC1 6.21 mm to (190.5, 144.8)
Routing:
- net Net-(D1-A): track 8.25 -> 2.36 mm
- net GND: track 75.9 -> 72.1 mm
- net Net-(D1-K): track 2.58 -> 0.87 mm
Other:
- board text added: "SDMAY24-21"
- board text removed: "REV 5A"

Commit message: update
Parts:
- removed C10, C13: 1uf - CC0805KKX5R8BB105, Capacitor_SMD:C_0805_2012Metric
- removed C14: 0.01uf - CC0805KRX7R9BB103, Capacitor_SMD:C_0805_2012Metric
- removed C15: 10uf - CC0805KKX5R8BB106, Capacitor_SMD:C_0805_2012Metric
- removed C16, C17: 0.1uf - CC0805KRX7R9BB104, Capacitor_SMD:C_0805_2012Metric
- removed D3, D4: LED - 17-215SURC/S530-A2/TR8, LED_SMD:LED_1206_3216Metric
- removed H1: MICROMOD-Standoff, MicroMod-Sparkfun:MicroMod-Standoff
- removed IC** (x4): SOIC127P600X175-8N (SRAM), SeniorDesign:SOIC127P600X175-8N (SRAM)
- removed IC**: QFP50P1200X1200X120-65N (ADC), SeniorDesign:QFP50P1200X1200X120-65N (ADC)
- removed J1: USB_B_Micro - 10118193-0001LF, strive_foot_prints:FCI_10118193-0001LF
- removed J2: Conn_01x02_Female, Connector_PinHeader_2.54mm:PinHeader_1x02_P2.54mm_Vertical
- removed J3, J6, J8: Conn_01x02_Male, Connector_PinHeader_2.54mm:PinHeader_1x02_P2.54mm_Vertical
- removed J4: Conn_01x03_Female, Connector_PinHeader_2.54mm:PinHeader_1x03_P2.54mm_Vertical
- removed R10, R12, R13, R7, R8, R9: 10k - RC0805FR-0710KL, Resistor_SMD:R_0805_2012Metric
- removed R11, R14: 82 - 0805W8F820JT5E, Resistor_SMD:R_0805_2012Metric
- removed R16, R5, R6: 10k, Resistor_SMD:R_0805_2012Metric
- removed R2: 12K 1% - 0805W8F1202T5E, Resistor_SMD:R_0805_2012Metric
- removed SW1: SW_Push - SKQGADE010, strive_foot_prints:SW4-SMD-5.2X5.2X1.5MM
- removed U1: FT232H, Package_DFN_QFN:QFN-48-1EP_8x8mm_P0.5mm_EP6.2x6.2mm
- removed U2, U3: SN74LVC1G125DCKR, strive_foot_prints:SOT65P210X110-5N
- removed U4: MCP1319MT-29LE-OT, Caravel_Board:PoR_5_SOT23
- removed U5, U6: TAR5SxxU_SOT353F, Caravel_Board:SOT-353F
- removed U7: W25Q32FVSS, strive_foot_prints:SOIC127P790X216-8N
- removed U8: caravel-M.2-card, MicroMod-Sparkfun:M.2-CONNECTOR-E
- removed X1: DSC6001_10MHZ, strive_foot_prints:DSC6001JE1A-010.0000
- removed Y1: CSTNE12M0GH5L000R0, strive_foot_prints:CSTNE12M0GH5L000R0
- added C1: 0.1uf - CC0805KRX7R9BB104, Capacitor_SMD:C_0805_2012Metric, F.Cu at (175.3, 125.4)
- added C2: 0.1uf - CC0805KRX7R9BB104, Capacitor_SMD:C_0805_2012Metric, F.Cu at (175.3, 112.7)
- added C3: 0.1uf - CC0805KRX7R9BB104, Capacitor_SMD:C_0805_2012Metric, F.Cu at (175.3, 99.1)
- added C4: 0.1uf - CC0805KRX7R9BB104, Capacitor_SMD:C_0805_2012Metric, F.Cu at (175.3, 87.3)
- added C5: 0.1uf - CC0805KRX7R9BB104, Capacitor_SMD:C_0805_2012Metric, F.Cu at (157.5, 68.6)
- added IC2: ADS1178IPAPT, SeniorDesign:QFP50P1200X1200X120-65N, F.Cu at (129.5, 114.3)
- added IC3: 23K256T-I_SN, SeniorDesign:SOIC127P600X175-8N, F.Cu at (162.6, 84.0)
- added IC4: 23K256T-I_SN, SeniorDesign:SOIC127P600X175-8N, F.Cu at (162.6, 96.7)
- added IC5: 23K256T-I_SN, SeniorDesign:SOIC127P600X175-8N, F.Cu at (162.6, 109.2)
- added IC6: 23K256T-I_SN, SeniorDesign:SOIC127P600X175-8N, F.Cu at (162.6, 121.9)
- J10: footprint Connector_PinHeader_2.54mm:PinHeader_1x27_P2.54mm_Vertical -> Connector_PinHeader_2.54mm:PinHeader_1x28_P2.54mm_Vertical
- J11: footprint Connector_PinHeader_2.54mm:PinHeader_1x20_P2.54mm_Vertical -> Connector_PinHeader_2.54mm:PinHeader_1x28_P2.54mm_Vertical
- moved IC1 94.5 mm to (134.2, 68.9), turned to 180 degrees
- moved J11 58.2 mm to (183.6, 132.0)
- moved J7 58.2 mm to (167.3, 132.7)
- moved TP2 58.2 mm to (178.1, 133.0)
- moved J10 58.2 mm to (111.1, 63.5)
- moved TP1 58.2 mm to (119.4, 132.3)
Connections:
- IC1 pad 13: unconnected-(IC1-GND-Pad13) -> GND
- IC1 pad 14: unconnected-(IC1-RSTSEL-Pad14) -> GND
- IC1 pad 17: unconnected-(IC1-~{RESET}-Pad17) -> ~{RST}
- IC1 pad 18: unconnected-(IC1-VREF-Pad18) -> Vref
- IC1 pad 3: unconnected-(IC1-VDD-Pad3) -> vddio
- IC1 pad 5: unconnected-(IC1-~{SYNC}-Pad5) -> GND
Routing:
- net vdda: track 379.7 -> 2.54 mm, vias 20 -> 0
- net vccd: track 263.7 -> 0.00 mm, vias 10 -> 0
- net GND: track 72.1 -> 294.5 mm, vias 18 -> 8
- net mprj_io[6]_ser_tx: track 150.5 -> 0.00 mm, vias 6 -> 0
- net mprj_io[5]_ser_rx: track 147.8 -> 0.00 mm, vias 7 -> 0
- net USB_SO_RXD: track 131.3 -> 0.00 mm, vias 5 -> 0
- net USB_SCK_TXD: track 131.2 -> 0.00 mm, vias 5 -> 0
- net USB_SI: track 94.0 -> 0.00 mm, vias 2 -> 0
- net USB_CS1: track 93.8 -> 0.00 mm, vias 4 -> 0
- net ~{RST}: track 82.2 -> 0.00 mm, vias 3 -> 0
- net gpio: track 78.2 -> 0.00 mm, vias 5 -> 0
- net vdda2: track 77.8 -> 0.00 mm, vias 4 -> 0
- net ~{MR}: track 76.8 -> 0.00 mm, vias 4 -> 0
- net mprj_io[0]: track 70.9 -> 0.00 mm, vias 2 -> 0
- net mprj_io[37]: track 68.4 -> 0.00 mm
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Other:
- board text removed: "1"
- board text removed: "Caravel"
- board text removed: "Display"
- board text removed: "M.2"
- board text removed: "MEMORY"
- board text removed: "Power"
- board text removed: "RESET"
- board text removed: "RX"
- board text removed: "SDMAY24-21"

Commit message: update again
Parts:
- removed C5: 0.1uf - CC0805KRX7R9BB104, Capacitor_SMD:C_0805_2012Metric
- IC2: value ADS1178IPAPT -> MCP3464T-E_NC; footprint SeniorDesign:QFP50P1200X1200X120-65N -> SeniorDesign:QFN40P300X300X60-21N-D
- moved IC2 2.30 mm to (129.5, 112.0)
Connections:
- IC1 pad 1: unconnected-(IC1-VOUT1-Pad1) -> mprj_io[29]
- IC1 pad 10: unconnected-(IC1-VOUT6-Pad10) -> mprj_io[32]
- IC1 pad 11: unconnected-(IC1-VOUT5-Pad11) -> mprj_io[37]
- IC1 pad 12: unconnected-(IC1-VOUT4-Pad12) -> mprj_io[36]
- IC1 pad 15: unconnected-(IC1-~{LDAC}-Pad15) -> mprj_io[35]
- IC1 pad 16: unconnected-(IC1-SDO-Pad16) -> mprj_io[1]_SDO
- IC1 pad 18: Vref -> vddio
- IC1 pad 19: unconnected-(IC1-VOUT3-Pad19) -> mprj_io[34]
- IC1 pad 2: unconnected-(IC1-VOUT0-Pad2) -> mprj_io[30]
- IC1 pad 20: unconnected-(IC1-VOUT2-Pad20) -> mprj_io[33]
- IC1 pad 4: unconnected-(IC1-VLOGIC-Pad4) -> vccd1
- IC1 pad 6: unconnected-(IC1-SCLK-Pad6) -> Caravel_SCK
- IC1 pad 7: unconnected-(IC1-SDI-Pad7) -> mprj_io[2]_SDI
- IC1 pad 8: unconnected-(IC1-GAIN-Pad8) -> vccd1
- IC1 pad 9: unconnected-(IC1-VOUT7-Pad9) -> mprj_io[31]
- IC2 pad 1: unconnected-(IC2-AINP2-Pad1) -> GND
- IC2 pad 10: GND -> mprj_io[15]
- IC2 pad 11: GND -> Caravel_CSB
- IC2 pad 12: GND -> Caravel_SCK
- IC2 pad 13: unconnected-(IC2-DOUT8-Pad13) -> mprj_io[2]_SDI
- IC2 pad 14: unconnected-(IC2-DOUT7-Pad14) -> mprj_io[1]_SDO
- IC2 pad 15: unconnected-(IC2-DOUT6-Pad15) -> GND
- IC2 pad 16: unconnected-(IC2-DOUT5-Pad16) -> GND
- IC2 pad 17: unconnected-(IC2-DOUT4-Pad17) -> GND
- IC2 pad 18: unconnected-(IC2-DOUT3-Pad18) -> vccd1
- IC2 pad 19: unconnected-(IC2-DOUT2-Pad19) -> vddio
- IC2 pad 2: unconnected-(IC2-AINN2-Pad2) -> vddio
- IC2 pad 20: unconnected-(IC2-DOUT1-Pad20) -> GND
- IC2 pad 3: unconnected-(IC2-AINP1-Pad3) -> mprj_io[22]
- IC2 pad 4: unconnected-(IC2-AINN1-Pad4) -> mprj_io[21]
- IC2 pad 5: vddio -> mprj_io[20]
- IC2 pad 6: GND -> mprj_io[19]
- IC2 pad 7: GND -> mprj_io[18]
- IC2 pad 8: GND -> mprj_io[17]
- IC2 pad 9: GND -> mprj_io[16]
- J10 pad 7: vdda -> vddio
- J11 pad 13: USB_SO_RXD -> mprj_io[2]_SDI
- J11 pad 14: USB_SI -> mprj_io[1]_SDO
- J11 pad 22: vccd -> vccd1
- J11 pad 23: vccd -> vccd1
- J11 pad 24: vccd -> vccd1
Routing:
- net vddio: track 0.00 -> 127.1 mm, vias 0 -> 6
- net mprj_io[1]_SDO: track 0.00 -> 110.0 mm, vias 0 -> 3
- net vccd1: track 0.00 -> 107.2 mm, vias 0 -> 4
- net mprj_io[2]_SDI: track 0.00 -> 105.7 mm, vias 0 -> 6
- net Caravel_CSB: track 76.7 -> 162.5 mm, vias 4 -> 7
- net Caravel_SCK: track 77.5 -> 150.8 mm, vias 4 -> 8
- net mprj_io[31]: track 0.00 -> 58.5 mm, vias 0 -> 1
- net mprj_io[32]: track 0.00 -> 54.1 mm, vias 0 -> 1
- net mprj_io[30]: track 0.00 -> 51.5 mm, vias 0 -> 1
- net mprj_io[29]: track 0.00 -> 50.1 mm, vias 0 -> 1
- net mprj_io[15]: track 0.00 -> 26.1 mm, vias 0 -> 1
- net mprj_io[33]: track 0.00 -> 24.1 mm
- net mprj_io[16]: track 0.00 -> 24.0 mm, vias 0 -> 1
- net mprj_io[17]: track 0.00 -> 22.3 mm, vias 0 -> 1
- net ~{RST}: track 0.00 -> 21.8 mm, vias 0 -> 1
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Other:
- board text added: "SDMAY24-21"
- board text added: "Yuwei Jonathan Sam Haris"

Commit message: update
Parts:
- added J1: SJ-63062A, SeniorDesign:CUI_SJ-63062A, F.Cu at (76.2, 68.6)
- added J10: Conn_01x27_Female, Connector_PinHeader_2.54mm:PinHeader_1x27_P2.54mm_Vertical, F.Cu at (-12.3, 2.98)
- added J11: Conn_01x20_Female, Connector_PinHeader_2.54mm:PinHeader_1x20_P2.54mm_Vertical, F.Cu at (-7.62, 2.98)
- added J2: SJ-63062A, SeniorDesign:CUI_SJ-63062A, F.Cu at (114.3, 167.6)
- added J7: Conn_01x06_Female, Connector_PinHeader_2.54mm:PinHeader_1x06_P2.54mm_Vertical, F.Cu at (-7.62, 55.9)
Connections:
- IC2 pad 3: mprj_io[22] -> Net-(IC2-CH0)

Commit message: update
Parts:
- removed the J10 at (-12.3, 2.98)
- removed the J11 at (-7.62, 2.98)
- removed the J7 at (-7.62, 55.9)
- moved J2 91.6 mm to (133.0, 78.0), turned to -90 degrees
- moved C2 85.1 mm to (251.1, 74.0), turned to 0 degrees
- moved C4 76.2 mm to (251.1, 79.5), turned to 0 degrees
- moved J1 74.9 mm to (150.5, 78.0), turned to -90 degrees
- moved C1 72.6 mm to (226.6, 74.0), turned to 0 degrees
- moved IC6 56.7 mm to (215.1, 100.6), turned to 0 degrees
- moved C3 54.9 mm to (226.6, 79.5), turned to 0 degrees
- moved IC5 54.7 mm to (215.1, 94.2), turned to 0 degrees
- moved IC4 53.3 mm to (215.1, 87.7), turned to 0 degrees
- moved IC3 52.6 mm to (215.1, 81.3), turned to 0 degrees
- moved IC1 32.1 mm to (133.0, 101.0)
- moved IC2 4.39 mm to (132.7, 109.0)
Connections:
- IC1 pad 1: mprj_io[29] -> unconnected-(IC1-VOUT1-Pad1)
- IC1 pad 10: mprj_io[32] -> Net-(IC1-VOUT6)
- IC1 pad 11: mprj_io[37] -> unconnected-(IC1-VOUT5-Pad11)
- IC1 pad 12: mprj_io[36] -> unconnected-(IC1-VOUT4-Pad12)
- IC1 pad 15: mprj_io[35] -> unconnected-(IC1-~{LDAC}-Pad15)
- IC1 pad 19: mprj_io[34] -> unconnected-(IC1-VOUT3-Pad19)
- IC1 pad 2: mprj_io[30] -> unconnected-(IC1-VOUT0-Pad2)
- IC1 pad 20: mprj_io[33] -> unconnected-(IC1-VOUT2-Pad20)
- IC1 pad 9: mprj_io[31] -> unconnected-(IC1-VOUT7-Pad9)
- IC2 pad 10: mprj_io[15] -> unconnected-(IC2-CH7-Pad10)
- IC2 pad 16: GND -> mprj_io[14]
- IC2 pad 6: mprj_io[19] -> unconnected-(IC2-CH3-Pad6)
- IC2 pad 7: mprj_io[18] -> unconnected-(IC2-CH4-Pad7)
- IC2 pad 8: mprj_io[17] -> unconnected-(IC2-CH5-Pad8)
- IC2 pad 9: mprj_io[16] -> unconnected-(IC2-CH6-Pad9)
- J2 pad 1: unconnected-(J2-Pad1) -> Net-(IC1-VOUT6)
Routing:
- net GND: track 296.8 -> 74.8 mm, vias 9 -> 4
- net Caravel_CSB: track 162.5 -> 0.00 mm, vias 7 -> 0
- net Caravel_SCK: track 150.8 -> 0.00 mm, vias 8 -> 0
- net mprj_io[2]_SDI: track 105.7 -> 0.00 mm, vias 6 -> 0
- net vdda1: track 98.3 -> 0.00 mm, vias 4 -> 0
- net vddio: track 127.1 -> 42.4 mm, vias 6 -> 1
- net Caravel_D1: track 83.3 -> 0.00 mm, vias 4 -> 0
- net Caravel_D0: track 81.1 -> 0.00 mm, vias 4 -> 0
- net ~{MEM_HOLD}: track 80.4 -> 0.00 mm, vias 4 -> 0
- net mprj_io[31]: track 58.5 -> 0.00 mm, vias 1 -> 0
- net mprj_io[32]: track 54.1 -> 0.00 mm, vias 1 -> 0
- net mprj_io[30]: track 51.5 -> 0.00 mm, vias 1 -> 0
- net mprj_io[29]: track 50.1 -> 0.00 mm, vias 1 -> 0
- net mprj_io[1]_SDO: track 110.0 -> 62.8 mm, vias 3 -> 1
- net vccd1: track 107.2 -> 79.5 mm, vias 4 -> 3
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Other:
- board text removed: "CS"
- board text removed: "SCK"
- board text removed: "SDMAY24-21"
- board text removed: "SI"
- board text removed: "SO"
- board text removed: "Yuwei Jonathan Sam Haris"
- board text removed: "~{HOLD}"
- board text removed: "~{WP}"

Commit message: update 4/5
Parts:
- added IC7: MCP3464T-E_NC, SeniorDesign:QFN40P300X300X60-21N-D, F.Cu at (124.3, 119.0)
- added VR1: 3360Y-1-103LF, SeniorDesign:3360Y1103LF, F.Cu at (138.5, 128.0)
- added VR2: 3360Y-1-103LF, SeniorDesign:3360Y1103LF, F.Cu at (148.2, 128.0)
- added VR3: 3360Y-1-103LF, SeniorDesign:3360Y1103LF, F.Cu at (138.5, 119.0)
- added VR4: 3360Y-1-103LF, SeniorDesign:3360Y1103LF, F.Cu at (148.2, 119.0)
- moved C2 87.3 mm to (173.5, 114.0)
- moved C4 80.6 mm to (173.5, 101.5)
- moved C1 71.2 mm to (173.5, 121.5)
- moved C3 59.8 mm to (173.4, 107.0)
- moved IC6 59.7 mm to (160.5, 124.7), turned to 180 degrees
- moved IC5 59.4 mm to (160.5, 117.5), turned to 180 degrees
- moved IC4 59.1 mm to (160.5, 110.3), turned to 180 degrees
- moved IC3 58.8 mm to (160.5, 103.1), turned to 180 degrees
- moved IC2 0.30 mm to (133.0, 109.0)
Connections:
- IC2 pad 16: mprj_io[14] -> mprj_io[21]
- IC2 pad 4: mprj_io[21] -> mprj_io[23]
- IC2 pad 5: mprj_io[20] -> mprj_io[22]
Routing:
- net GND: track 74.8 -> 249.1 mm, vias 4 -> 15
- net +3.3V: track 0.00 -> 143.8 mm, vias 0 -> 17
- net Caravel_CSB: track 0.00 -> 123.9 mm, vias 0 -> 2
- net Caravel_SCK: track 0.00 -> 113.3 mm, vias 0 -> 9
- net mprj_io[2]_SDI: track 0.00 -> 93.0 mm, vias 0 -> 4
- net vddio: track 42.4 -> 99.9 mm, vias 1 -> 7
- net Net-(IC2-CH0): track 0.00 -> 54.0 mm, vias 0 -> 3
- net mprj_io[1]_SDO: track 62.8 -> 113.2 mm, vias 1 -> 8
- net Caravel_D0: track 0.00 -> 46.9 mm
- net ~{MEM_HOLD}: track 0.00 -> 42.4 mm, vias 0 -> 4
- net Caravel_D1: track 0.00 -> 40.7 mm, vias 0 -> 4
- net vccd1: track 79.5 -> 119.5 mm, vias 3 -> 11
- net mprj_io[21]: track 0.00 -> 33.9 mm, vias 0 -> 1
- net Net-(IC7-CH5): track 0.00 -> 33.7 mm, vias 0 -> 1
- net Net-(IC7-CH4): track 0.00 -> 24.5 mm, vias 0 -> 1
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
Commit message: last update
Parts:
- added IC8: LMV1032UP-06_NOPB, SeniorDesign:BGA4C50P2X2_115X115X40, F.Cu at (135.2, 87.8)
- J11: value Conn_01x20_Female -> Conn_01x28_Pin
- moved J2 32.0 mm to (165.0, 78.1)
- moved IC1 29.1 mm to (127.0, 72.5)
- moved IC2 22.5 mm to (126.4, 87.5), turned to 180 degrees
- moved IC7 10.2 mm to (126.5, 129.0), turned to 180 degrees
- moved C3 6.21 mm to (175.1, 113.0)
- moved C2 5.71 mm to (175.1, 119.5)
- moved IC3 5.43 mm to (162.8, 108.0), turned to 0 degrees
- moved C4 5.23 mm to (175.1, 106.5)
- moved IC4 4.81 mm to (162.8, 114.5), turned to 0 degrees
- moved C1 4.76 mm to (175.1, 126.0)
- moved IC5 4.25 mm to (162.8, 121.1), turned to 0 degrees
- moved IC6 3.72 mm to (162.8, 127.6), turned to 0 degrees
- moved J1 3.50 mm to (147.0, 78.1)
- moved VR1 1.00 mm to (139.5, 128.0)
- moved VR2 1.00 mm to (149.2, 128.0)
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Connections:
- net USB_CS1 renamed /mprj_io[3]_CSB
- net USB_SCK_TXD renamed /mprj_io[4]_SCK
- net gpio renamed /gpio
- net mprj_io[0] renamed /mprj_io[0]
- net mprj_io[5]_ser_rx renamed /mprj_io[5]_ser_rx
- net mprj_io[6]_ser_tx renamed /mprj_io[6]_ser_tx
- net vccd2 renamed /vccd2
- net vdda renamed +3V3
- net vdda1 renamed /vdda1
- net vdda2 renamed /vdda2
- net xclk renamed /xclk
- IC1 pad 14: GND -> mprj_io[35]
- IC1 pad 16: mprj_io[1]_SDO -> mprj_io[34]
- IC1 pad 5: GND -> unconnected-(IC1-~{SYNC}-Pad5)
- IC1 pad 6: Caravel_SCK -> mprj_io[36]
- IC1 pad 7: mprj_io[2]_SDI -> mprj_io[37]
- IC2 pad 11: Caravel_CSB -> mprj_io[31]
- IC2 pad 12: Caravel_SCK -> mprj_io[30]
- IC2 pad 13: mprj_io[2]_SDI -> mprj_io[29]
- IC2 pad 14: mprj_io[1]_SDO -> mprj_io[28]
- IC2 pad 16: mprj_io[21] -> mprj_io[27]
- IC2 pad 4: mprj_io[23] -> mprj_io[33]
- IC2 pad 5: mprj_io[22] -> mprj_io[32]
- IC3 pad 1: Caravel_CSB -> SRAM_CS0
- IC3 pad 2: Caravel_D1 -> SRAM_SO0
- IC3 pad 5: Caravel_D0 -> SRAM_SI
- IC3 pad 6: Caravel_SCK -> SRAM_SCK
- IC3 pad 7: ~{MEM_HOLD} -> mprj_io[11]
- IC4 pad 1: Caravel_CSB -> SRAM_CS0
- IC4 pad 2: Caravel_D1 -> SRAM_SO1
- IC4 pad 5: Caravel_D0 -> SRAM_SI
- IC4 pad 6: Caravel_SCK -> SRAM_SCK
- IC4 pad 7: ~{MEM_HOLD} -> mprj_io[11]
- IC5 pad 1: Caravel_CSB -> SRAM_CS1
- IC5 pad 2: Caravel_D1 -> SRAM_SO0
- IC5 pad 5: Caravel_D0 -> SRAM_SI
- IC5 pad 6: Caravel_SCK -> SRAM_SCK
- IC5 pad 7: ~{MEM_HOLD} -> mprj_io[11]
- IC6 pad 1: Caravel_CSB -> SRAM_CS1
- IC6 pad 2: Caravel_D1 -> SRAM_SO1
- IC6 pad 5: Caravel_D0 -> SRAM_SI
- IC6 pad 6: Caravel_SCK -> SRAM_SCK
- IC6 pad 7: ~{MEM_HOLD} -> mprj_io[11]
- IC7 pad 11: Caravel_CSB -> mprj_io[17]
- IC7 pad 12: Caravel_SCK -> mprj_io[16]
- IC7 pad 13: mprj_io[2]_SDI -> mprj_io[15]
- IC7 pad 14: mprj_io[1]_SDO -> mprj_io[14]
- J1 pad 1: Net-(IC2-CH0) -> Net-(IC8-INPUT)
- J11 pad 13: mprj_io[2]_SDI -> /mprj_io[2]_SDI
- J11 pad 14: mprj_io[1]_SDO -> /mprj_io[1]_SDO
- J11 pad 2: mprj_io[13] -> SRAM_SI
- J11 pad 22: vccd1 -> +1V8
- J11 pad 23: vccd1 -> +1V8
- J11 pad 3: mprj_io[12] -> SRAM_SCK
- J11 pad 5: mprj_io[10] -> SRAM_SO1
- J11 pad 6: mprj_io[9] -> SRAM_CS1
- J11 pad 7: mprj_io[8] -> SRAM_SO0
- J11 pad 8: mprj_io[7] -> SRAM_CS0
Routing:
- net Caravel_CSB: track 123.9 -> 0.00 mm, vias 2 -> 0
- net Caravel_SCK: track 113.3 -> 0.00 mm, vias 9 -> 0
- net mprj_io[1]_SDO: track 113.2 -> 0.00 mm, vias 8 -> 0
- net mprj_io[2]_SDI: track 93.0 -> 0.00 mm, vias 4 -> 0
- net +3.3V: track 143.8 -> 54.5 mm, vias 17 -> 0
- net mprj_io[11]: track 0.00 -> 50.4 mm, vias 0 -> 4
- net SRAM_SO0: track 0.00 -> 49.5 mm, vias 0 -> 4
- net Caravel_D0: track 46.9 -> 0.00 mm
- net SRAM_SO1: track 0.00 -> 46.8 mm, vias 0 -> 4
- net Net-(IC2-CH0): track 54.0 -> 7.31 mm, vias 3 -> 0
- net SRAM_SCK: track 0.00 -> 45.9 mm, vias 0 -> 4
- net SRAM_CS0: track 0.00 -> 45.3 mm, vias 0 -> 2
- net vddio: track 99.9 -> 142.5 mm, vias 7 -> 9
- net ~{MEM_HOLD}: track 42.4 -> 0.00 mm, vias 4 -> 0
- net SRAM_SI: track 0.00 -> 42.2 mm, vias 0 -> 4
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