File: breakout_board_PCB/BreakoutBoardPCB/BreakoutBoardPCB.kicad_pcb (KiCad board)
At the start: 2 copper layers, 76.2 x 73.8 mm, 23 parts, among them IC1 AD5676BRUZ, IC2 MCP3464T-E_NC, IC3 23K256T-I_SN, IC4 23K256T-I_SN, IC5 23K256T-I_SN, IC6 23K256T-I_SN, IC7 MCP3464T-E_NC, IC8 LMV1032UP-06_NOPB, J1 SJ-63062A, J10 Conn_01x27_Female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

Commit message: update
Connections:
- J11 pad 26: +3V3 -> +3.3V
- J11 pad 27: +3V3 -> +3.3V
Routing:
- net +3.3V: track 54.5 -> 174.8 mm, vias 0 -> 1
- net GND: track 272.7 -> 276.2 mm
- net +3V3: track 2.54 -> 0.00 mm
- net +1V8: track 0.00 -> 2.54 mm
Other:
- board text added: "Haris Khan, Jonathan Hess"
- board text added: "Yuwei Tan, Sam Heikens"
- board text added: "sdmay24-21"
Changed lines of the file:
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@@
 			(disableapertmacros no)
 			(usegerberextensions yes)
-			(usegerberattributes no)
+			(usegerberattributes yes)
 			(usegerberadvancedattributes no)
 			(creategerberjobfile no)
@@
 			(drillshape 0)
 			(scaleselection 1)
-			(outputdirectory "gerbers/")
+			(outputdirectory "/Users/tanyuwei/ASIC-GuitarPedal/breakout_board_PCB/BreakoutBoardPCB/newgerbers/")
 		)
 	)
@@
 	(net 77 "/mprj_io[5]_ser_rx")
 	(net 78 "/mprj_io[4]_SCK")
-	(net 79 "+3V3")
-	(net 80 "/vdda2")
-	(net 81 "/mprj_io[6]_ser_tx")
-	(net 82 "/gpio")
-	(net 83 "/mprj_io[1]_SDO")
-	(net 84 "/mprj_io[0]")
-	(net 85 "/vdda1")
-	(net 86 "/vccd2")
+	(net 79 "/vdda2")
+	(net 80 "/mprj_io[6]_ser_tx")
+	(net 81 "/gpio")
+	(net 82 "/mprj_io[1]_SDO")
+	(net 83 "/mprj_io[0]")
+	(net 84 "/vdda1")
+	(net 85 "/vccd2")
 	(footprint "SeniorDesign:SOIC127P600X175-8N"
 		(layer "F.Cu")
@@
 		)
 		(fp_text user "${REFERENCE}"
-			(at 0 34.29 270)
+			(at 0 34.29 -90)
 			(layer "F.Fab")
 			(effects
@@
 			(layers "*.Cu" "*.Mask")
 			(remove_unused_layers no)
-			(net 81 "/mprj_io[6]_ser_tx")
+			(net 80 "/mprj_io[6]_ser_tx")
 			(pinfunction "Pin_9")
 			(pintype "passive")
@@
 			(layers "*.Cu" "*.Mask")
 			(remove_unused_layers no)
-			(net 83 "/mprj_io[1]_SDO")
+			(net 82 "/mprj_io[1]_SDO")
 			(pinfunction "Pin_14")
 			(pintype "passive")
@@
 			(layers "*.Cu" "*.Mask")
 			(remove_unused_layers no)
-			(net 84 "/mprj_io[0]")
+			(net 83 "/mprj_io[0]")
 			(pinfunction "Pin_15")
 			(pintype "passive")
@@
 			(layers "*.Cu" "*.Mask")
 			(remove_unused_layers no)
-			(net 85 "/vdda1")
+			(net 84 "/vdda1")
 			(pinfunction "Pin_16")
 			(pintype "passive")
@@
 			(layers "*.Cu" "*.Mask")
 			(remove_unused_layers no)
-			(net 82 "/gpio")
+			(net 81 "/gpio")
 			(pinfunction "Pin_20")
 			(pintype "passive")
@@
 			(layers "*.Cu" "*.Mask")
 			(remove_unused_layers no)
-			(net 86 "/vccd2")
+			(net 85 "/vccd2")
 			(pinfunction "Pin_21")
 			(pintype "passive")
@@
 			(layers "*.Cu" "*.Mask")
 			(remove_unused_layers no)
-			(net 80 "/vdda2")
+			(net 79 "/vdda2")
 			(pinfunction "Pin_25")
 			(pintype "passive")
@@
 			(layers "*.Cu" "*.Mask")
 			(remove_unused_layers no)
-			(net 79 "+3V3")
+			(net 28 "+3.3V")
 			(pinfunction "Pin_26")
 			(pintype "passive")
@@
 			(layers "*.Cu" "*.Mask")
 			(remove_unused_layers no)
-			(net 79 "+3V3")
+			(net 28 "+3.3V")
 			(pinfunction "Pin_27")
 			(pintype "passive")
@@
 		)
 	)
+	(gr_text "Haris Khan, Jonathan Hess"
+		(at 139.5 102.5 0)
+		(layer "F.SilkS")
+		(effects
+			(font
+				(size 1 1)
+				(thickness 0.15)
+			)
+			(justify left bottom)
+		)
+	)
 	(gr_text "IO[6]"
 		(at 179.809207 111.785601 0)
@@
 		)
 	)
+	(gr_text "Yuwei Tan, Sam Heikens"
+		(at 140.5 100.5 0)
+		(layer "F.SilkS")
+		(effects
+			(font
+				(size 1 1)
+				(thickness 0.15)
+			)
+			(justify left bottom)
+		)
+	)
 	(gr_text "IO[4]"
 		(at 179.783807 106.756401 0)
@@
 		)
 	)
+	(gr_text "sdmay24-21"
+		(at 144 98.5 0)
+		(layer "F.SilkS")
+		(effects
+			(font
+				(size 1 1)
+				(thickness 0.15)
+			)
+			(justify left bottom)
+		)
+	)
 	(gr_text "IO[22]"
 		(at 115.521807 109.144001 0)
@@
 	)
 	(segment
+		(start 126.4 87.5)
+		(end 126 87.9)
+		(width 0.1524)
+		(layer "F.Cu")
+		(net 1)
+	)
+	(segment
 		(start 115.125 70.875)
 		(end 115 71)
@@
 	)
 	(segment
+		(start 126 87.9)
+		(end 126 89)
+		(width 0.1524)
+		(layer "F.Cu")
+		(net 1)
+	)
+	(segment
 		(start 124.9 89.423156)
 		(end 124.9 88.3)
@@
 	)
 	(segment
+		(start 126.5 129)
+		(end 127.3 129.8)
+		(width 0.1524)
+		(layer "F.Cu")
+		(net 1)
+	)
+	(segment
 		(start 127.5 90)
 		(end 127.2 89.7)
@@
 	)
 	(segment
+		(start 127.3 129.8)
+		(end 127.3 130.5)
+		(width 0.1524)
+		(layer "F.Cu")
+		(net 1)
+	)
+	(segment
 		(start 155.5 123)
 		(end 155.5 129.5)
@@
 	)
 	(segment
+		(start 139.5 119)
+		(end 139.5 128)
+		(width 0.1524)
+		(layer "F.Cu")
+		(net 28)
+	)
+	(segment
 		(start 173.83 125.73)
 		(end 174.1 126)
@@
 	)
 	(segment
+		(start 175.004001 68.504001)
+		(end 183.568407 68.504001)
+		(width 0.1524)
+		(layer "F.Cu")
+		(net 28)
+	)
+	(segment
 		(start 173.73 112.63)
 		(end 174.1 113)
@@
 	)
 	(segment
+		(start 175 68.5)
+		(end 175.004001 68.504001)
+		(width 0.1524)
+		(layer "F.Cu")
+		(net 28)
+	)
+	(segment
 		(start 174.1 126)
 		(end 174.1 119.5)
@@
 	)
 	(segment
+		(start 174.1 68.9)
+		(end 174.5 68.5)
+		(width 0.1524)
+		(layer "F.Cu")
+		(net 28)
+	)
+	(segment
+		(start 149.1975 119)
+		(end 149.1975 128)
+		(width 0.1524)
+		(layer "F.Cu")
+		(net 28)
+	)
+	(segment
 		(start 165.5 125.73)
 		(end 173.83 125.73)
@@
 	)
 	(segment
+		(start 174.1 103.5)
+		(end 174.1 68.9)
+		(width 0.1524)
+		(layer "F.Cu")
+		(net 28)
+	)
+	(segment
 		(start 174.1 119.5)
 		(end 174.1 113)
@@
 	)
 	(segment
+		(start 174.1 106.5)
+		(end 174.1 103.5)
+		(width 0.1524)
+		(layer "F.Cu")
+		(net 28)
+	)
+	(segment
 		(start 165.5 106.08)
 		(end 173.68 106.08)
@@
 	)
 	(segment
+		(start 174.5 68.5)
+		(end 175 68.5)
+		(width 0.1524)
+		(layer "F.Cu")
+		(net 28)
+	)
+	(segment
 		(start 173.68 106.08)
 		(end 174.1 106.5)
@@
 		(net 28)
 	)
+	(via
+		(at 174.1 103.5)
+		(size 0.5)
+		(drill 0.25)
+		(layers "F.Cu" "B.Cu")
+		(net 28)
+	)
+	(segment
+		(start 155 116)
+		(end 155 104)
+		(width 0.1524)
+		(layer "B.Cu")
+		(net 28)
+	)
+	(segment
+		(start 155.5 103.5)
+		(end 174.1 103.5)
+		(width 0.1524)
+		(layer "B.Cu")
+		(net 28)
+	)
+	(segment
+		(start 155 104)
+		(end 155.5 103.5)
+		(width 0.1524)
+		(layer "B.Cu")
+		(net 28)
+	)
+	(segment
+		(start 139.5 119)
+		(end 139.5 116.5)
+		(width 0.1524)
+		(layer "B.Cu")
+		(net 28)
+	)
+	(segment
+		(start 183.568407 65.964001)
+		(end 183.568407 68.504001)
+		(width 0.1524)
+		(layer "B.Cu")
+		(net 28)
+	)
+	(segment
+		(start 149 116)
+		(end 155 116)
+		(width 0.1524)
+		(layer "B.Cu")
+		(net 28)
+	)
+	(segment
+		(start 140 116)
+		(end 149 116)
+		(width 0.1524)
+		(layer "B.Cu")
+		(net 28)
+	)
+	(segment
+		(start 139.5 116.5)
+		(end 140 116)
+		(width 0.1524)
+		(layer "B.Cu")
+		(net 28)
+	)
+	(segment
+		(start 149 116)
+		(end 149.1975 116.1975)
+		(width 0.1524)
+		(layer "B.Cu")
+		(net 28)
+	)
+	(segment
+		(start 149.1975 116.1975)
+		(end 149.1975 119)
+		(width 0.1524)
+		(layer "B.Cu")
+		(net 28)
+	)
 	(segment
 		(start 122 77)
@@
 	)
 	(segment
-		(start 183.568407 65.964001)
-		(end 183.568407 68.504001)
+		(start 183.568407 76.124001)
+		(end 183.568407 78.664001)
 		(width 0.1524)
 		(layer "B.Cu")
-		(net 79)
+		(net 74)
 	)
 	(zone
