File: breakout_board_PCB/BreakoutBoardPCB/BreakoutBoardPCB.kicad_pcb (KiCad board)
At the start: 2 copper layers, 76.2 x 73.8 mm, 23 parts, among them IC1 AD5676BRUZ, IC2 MCP3464T-E_NC, IC3 23K256T-I_SN, IC4 23K256T-I_SN, IC5 23K256T-I_SN, IC6 23K256T-I_SN, IC7 MCP3464T-E_NC, IC8 LMV1032UP-06_NOPB, J1 SJ-63062A, J10 Conn_01x27_Female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

Commit message: update
Connections:
- net Caravel_CSB renamed MEM_CS
- net Caravel_D0 renamed MEM_SI
- net Caravel_D1 renamed MEM_SO
- net Caravel_SCK renamed MEM_SCK
